File: Lion1_2.brd (EAGLE design)
At the start: 100 x 85.7 mm, 74 parts, among them IC1 MCP4822, IC2 MCP4822, IC3 MCP4822, IC4 REG1117, U7 2564-, U8 2564-

Commit message: v2
Connections:
- net N$24 renamed TX2
- net N$85 renamed RX2
- removed net 3V3: JP1.4, JP10.2, JP10.4, JP10.6
- net 3V3_7: now also JP15.1
- net 3V3_8: now also JP1.4, JP10.2, JP10.4, JP10.6
Routing:
- net 3V3: track 49.2 -> 0.00 mm
- net 3V3_7: track 61.0 -> 110.0 mm
- net 3V3_8: track 6.39 -> 49.6 mm, vias 0 -> 1
Changed lines of the file:
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@@
 <wire x1="83.4136" y1="36.068" x2="83.185" y2="35.8775" width="0.6096" layer="16"/>
-</signal>
-<signal name="3V3">
-<contactref element="JP1" pad="4"/>
-<contactref element="JP10" pad="6"/>
-<contactref element="JP10" pad="2"/>
-<contactref element="JP10" pad="4"/>
-<wire x1="4.4704" y1="32.3088" x2="4.4704" y2="29.8704" width="0.3048" layer="1"/>
-<wire x1="4.4704" y1="29.8704" x2="4.445" y2="29.845" width="0.3048" layer="1"/>
-<wire x1="4.4704" y1="32.3088" x2="4.445" y2="32.385" width="0.3048" layer="1"/>
-<wire x1="4.4704" y1="32.512" x2="4.4704" y2="34.8488" width="0.3048" layer="1"/>
-<wire x1="4.4704" y1="34.8488" x2="4.445" y2="34.925" width="0.3048" layer="1"/>
-<wire x1="4.4704" y1="32.512" x2="4.445" y2="32.385" width="0.3048" layer="1"/>
-<wire x1="16.4592" y1="2.4384" x2="18.3896" y2="4.3688" width="0.3048" layer="16"/>
-<wire x1="10.2616" y1="2.4384" x2="16.4592" y2="2.4384" width="0.3048" layer="16"/>
-<wire x1="9.5504" y1="3.1496" x2="10.2616" y2="2.4384" width="0.3048" layer="16"/>
-<wire x1="9.5504" y1="13.3096" x2="9.5504" y2="3.1496" width="0.3048" layer="16"/>
-<wire x1="5.2832" y1="13.3096" x2="9.5504" y2="13.3096" width="0.3048" layer="16"/>
-<wire x1="2.4384" y1="16.1544" x2="5.2832" y2="13.3096" width="0.3048" layer="16"/>
-<wire x1="2.4384" y1="29.7688" x2="2.4384" y2="16.1544" width="0.3048" layer="16"/>
-<wire x1="4.3688" y1="29.7688" x2="2.4384" y2="29.7688" width="0.3048" layer="16"/>
-<wire x1="18.3896" y1="4.3688" x2="18.415" y2="4.445" width="0.3048" layer="16"/>
-<wire x1="4.3688" y1="29.7688" x2="4.445" y2="29.845" width="0.3048" layer="16"/>
 </signal>
 <signal name="+5V">
@@
 <contactref element="U7" pad="34"/>
 </signal>
-<signal name="N$85">
+<signal name="RX2">
 <contactref element="U7" pad="36"/>
 <contactref element="JP15" pad="3"/>
@@
 <wire x1="57.2008" y1="27.5336" x2="57.15" y2="27.6225" width="0.3048" layer="1"/>
 </signal>
-<signal name="N$24">
+<signal name="TX2">
 <contactref element="JP15" pad="2"/>
 <contactref element="U7" pad="35"/>
@@
 <contactref element="U8" pad="4"/>
 <contactref element="R25" pad="2"/>
-<wire x1="8.2296" y1="14.6304" x2="8.2296" y2="18.3896" width="0.3048" layer="1"/>
-<wire x1="8.2296" y1="18.3896" x2="8.255" y2="18.415" width="0.3048" layer="1"/>
-<wire x1="8.2296" y1="14.6304" x2="8.255" y2="14.605" width="0.3048" layer="1"/>
 <wire x1="8.2296" y1="14.5288" x2="8.2296" y2="12.0904" width="0.3048" layer="1"/>
 <wire x1="8.2296" y1="12.0904" x2="8.255" y2="12.065" width="0.3048" layer="1"/>
 <wire x1="8.2296" y1="14.5288" x2="8.255" y2="14.605" width="0.3048" layer="1"/>
+<contactref element="JP10" pad="2"/>
+<contactref element="JP10" pad="4"/>
+<contactref element="JP10" pad="6"/>
+<wire x1="4.4704" y1="34.8488" x2="4.445" y2="34.925" width="0.3048" layer="1"/>
+<contactref element="JP1" pad="4"/>
+<wire x1="4.4704" y1="29.8704" x2="4.4704" y2="32.3088" width="0.3048" layer="1"/>
+<wire x1="4.4704" y1="32.3088" x2="4.445" y2="32.385" width="0.3048" layer="1"/>
+<wire x1="4.4704" y1="29.8704" x2="4.445" y2="29.845" width="0.3048" layer="1"/>
+<wire x1="4.4704" y1="32.512" x2="4.4704" y2="34.7472" width="0.3048" layer="1"/>
+<wire x1="4.4704" y1="34.7472" x2="4.445" y2="34.925" width="0.3048" layer="1"/>
+<wire x1="4.4704" y1="32.512" x2="4.445" y2="32.385" width="0.3048" layer="1"/>
+<wire x1="18.3896" y1="7.4168" x2="18.3896" y2="4.4704" width="0.3048" layer="1"/>
+<wire x1="18.3896" y1="4.4704" x2="18.415" y2="4.445" width="0.3048" layer="1"/>
+<via x="18.3896" y="7.4168" extent="1-16" drill="0.4064"/>
+<wire x1="8.255" y1="18.415" x2="1.905" y2="18.415" width="0.4064" layer="16"/>
+<wire x1="1.905" y1="18.415" x2="1.905" y2="29.845" width="0.4064" layer="16"/>
+<wire x1="1.905" y1="29.845" x2="4.445" y2="29.845" width="0.4064" layer="16"/>
+<wire x1="8.255" y1="18.415" x2="8.255" y2="14.605" width="0.4064" layer="1"/>
+<wire x1="8.255" y1="7.4295" x2="8.255" y2="12.065" width="0.4064" layer="16"/>
+<wire x1="8.255" y1="7.4295" x2="18.3896" y2="7.4295" width="0.4064" layer="16"/>
+<wire x1="18.3896" y1="7.4295" x2="18.3896" y2="7.4168" width="0.4064" layer="16"/>
 </signal>
 <signal name="3V3_7">
@@
 <wire x1="24.2824" y1="58.8264" x2="24.13" y2="59.055" width="0.3048" layer="16"/>
 <via x="24.6888" y="52.9336" extent="1-16" drill="0.4064"/>
+<contactref element="JP15" pad="1"/>
+<wire x1="45.72" y1="80.645" x2="28.575" y2="80.645" width="0.4064" layer="16"/>
+<wire x1="28.448" y1="83.82" x2="28.448" y2="80.772" width="0.3048" layer="16"/>
+<wire x1="27.7368" y1="84.2137" x2="28.448" y2="83.82" width="0.3048" layer="16"/>
+<wire x1="10.0584" y1="84.2137" x2="27.7368" y2="84.2137" width="0.3048" layer="16"/>
+<wire x1="9.3472" y1="83.82" x2="10.0584" y2="84.2137" width="0.3048" layer="16"/>
+<wire x1="9.3472" y1="75.5904" x2="9.3472" y2="83.82" width="0.3048" layer="16"/>
+<wire x1="8.3312" y1="75.5904" x2="9.3472" y2="75.5904" width="0.3048" layer="16"/>
+<wire x1="28.448" y1="80.772" x2="28.575" y2="80.645" width="0.3048" layer="16"/>
+<wire x1="8.3312" y1="75.5904" x2="8.255" y2="75.565" width="0.3048" layer="16"/>
 </signal>
 <signal name="N$9">

Commit message: some syslib functions, audio sample play command, 1 resistor added
Parts:
- added R30: 100K, SmartPrj:0204/7
Connections:
- net ADD: now also R30.1
- net GND8_1: now also R30.2
Routing:
- net ADD: track 31.3 -> 47.0 mm, vias 0 -> 1
- net GND8_1: track 148.0 -> 151.1 mm
Changed lines of the file:
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@@
 </element>
 <element name="R29" library="SmartPrj" package="0204V" value="" x="69.85" y="28.8925" rot="R90"/>
+<element name="R30" library="SmartPrj" package="0204/7" value="100K" x="42.2275" y="41.5925" rot="R90"/>
 </elements>
 <signals>
@@
 <wire x1="50.8" y1="28.6512" x2="50.8" y2="28.575" width="0.3048" layer="16"/>
 <wire x1="57.0992" y1="30.1752" x2="57.15" y2="30.1625" width="0.3048" layer="16"/>
+<contactref element="R30" pad="1"/>
+<wire x1="42.2656" y1="35.7632" x2="42.2656" y2="37.6936" width="0.3048" layer="1"/>
+<wire x1="40.64" y1="34.1376" x2="42.2656" y2="35.7632" width="0.3048" layer="1"/>
+<wire x1="40.64" y1="31.496" x2="40.64" y2="34.1376" width="0.3048" layer="1"/>
+<wire x1="40.7416" y1="31.3944" x2="40.64" y2="31.496" width="0.3048" layer="1"/>
+<wire x1="40.9448" y1="31.3944" x2="40.7416" y2="31.3944" width="0.3048" layer="1"/>
+<wire x1="46.5328" y1="31.3944" x2="40.9448" y2="31.3944" width="0.3048" layer="16"/>
+<wire x1="47.5488" y1="32.4104" x2="46.5328" y2="31.3944" width="0.3048" layer="16"/>
+<wire x1="48.8696" y1="32.4104" x2="47.5488" y2="32.4104" width="0.3048" layer="16"/>
+<wire x1="42.2656" y1="37.6936" x2="42.2275" y2="37.7825" width="0.3048" layer="1"/>
+<wire x1="48.8696" y1="32.4104" x2="48.895" y2="32.385" width="0.3048" layer="16"/>
+<via x="40.9448" y="31.3944" extent="1-16" drill="0.4064"/>
 </signal>
 <signal name="N$11">
@@
 <wire x1="30.48" y1="4.4704" x2="30.48" y2="4.445" width="0.3048" layer="16"/>
 <wire x1="10.8712" y1="4.4704" x2="10.795" y2="4.445" width="0.3048" layer="16"/>
+<contactref element="R30" pad="2"/>
+<wire x1="45.3136" y1="45.4152" x2="42.2656" y2="45.4152" width="0.3048" layer="16"/>
+<wire x1="42.2656" y1="45.4152" x2="42.2275" y2="45.4025" width="0.3048" layer="16"/>
+<wire x1="45.3136" y1="45.4152" x2="45.4025" y2="45.4025" width="0.3048" layer="16"/>
 </signal>
 <signal name="GND_1">
